File: Eagle files/LogicLab.brd (EAGLE design)
At the start: 139.7 x 91.4 mm, 122 parts, among them J1 1X4-BIG, J2 1X4-BIG, U1 AVR128DA48

Commit message: Version 1 - 18th May 2023
Parts:
- L2: value Amber -> Yellow
- L5: value Yellow -> Orange
Changed lines of the file:
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@@
 <attribute name="VALUE" x="19.685" y="13.97" size="1.27" layer="27" rot="R90"/>
 </element>
-<element name="L2" library="SparkFun-LED" package="LED5MM" value="Amber" x="133.35" y="55.88" smashed="yes">
+<element name="L2" library="SparkFun-LED" package="LED5MM" value="Yellow" x="133.35" y="55.88" smashed="yes">
 <attribute name="NAME" x="133.35" y="59.69" size="1.27" layer="25" ratio="10" align="bottom-center"/>
 <attribute name="VALUE" x="131.4704" y="50.2666" size="1.27" layer="27" ratio="10"/>
@@
 <attribute name="VALUE" x="125.73" y="18.415" size="1.27" layer="27"/>
 </element>
-<element name="L5" library="SparkFun-LED" package="LED5MM" value="Yellow" x="133.35" y="21.59" smashed="yes">
+<element name="L5" library="SparkFun-LED" package="LED5MM" value="Orange" x="133.35" y="21.59" smashed="yes">
 <attribute name="NAME" x="133.35" y="25.4" size="1.27" layer="25" ratio="10" align="bottom-center"/>
 <attribute name="VALUE" x="131.4704" y="15.9766" size="1.27" layer="27" ratio="10"/>

Commit message: Version 1 - 18th May 2023
Parts:
- L2: value Yellow -> Orange
- L5: value Orange -> Yellow
Changed lines of the file:
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@@
 <attribute name="VALUE" x="19.685" y="13.97" size="1.27" layer="27" rot="R90"/>
 </element>
-<element name="L2" library="SparkFun-LED" package="LED5MM" value="Yellow" x="133.35" y="55.88" smashed="yes">
+<element name="L2" library="SparkFun-LED" package="LED5MM" value="Orange" x="133.35" y="55.88" smashed="yes">
 <attribute name="NAME" x="133.35" y="59.69" size="1.27" layer="25" ratio="10" align="bottom-center"/>
 <attribute name="VALUE" x="131.4704" y="50.2666" size="1.27" layer="27" ratio="10"/>
@@
 <attribute name="VALUE" x="125.73" y="18.415" size="1.27" layer="27"/>
 </element>
-<element name="L5" library="SparkFun-LED" package="LED5MM" value="Orange" x="133.35" y="21.59" smashed="yes">
+<element name="L5" library="SparkFun-LED" package="LED5MM" value="Yellow" x="133.35" y="21.59" smashed="yes">
 <attribute name="NAME" x="133.35" y="25.4" size="1.27" layer="25" ratio="10" align="bottom-center"/>
 <attribute name="VALUE" x="131.4704" y="15.9766" size="1.27" layer="27" ratio="10"/>
