File: Eagle files/LogicLab.sch (EAGLE design)
At the start: 122 parts, among them J1 1X4-BIG, J2 1X4-BIG, U1 AVR128DA48

Commit message: Version 1 - 18th May 2023
Parts:
- L2: value Amber -> Yellow
- L5: value Yellow -> Orange
Changed lines of the file:
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@@
 <layer number="93" name="Pins" color="2" fill="1" visible="no" active="yes"/>
 <layer number="94" name="Symbols" color="4" fill="1" visible="yes" active="yes"/>
-<layer number="95" name="Names" color="7" fill="1" visible="yes" active="yes"/>
+<layer number="95" name="Names" color="7" fill="1" visible="no" active="yes"/>
 <layer number="96" name="Values" color="7" fill="1" visible="yes" active="yes"/>
 <layer number="97" name="Info" color="7" fill="1" visible="yes" active="yes"/>
@@
 <part name="JP7" library="adafruit" deviceset="PINHD-1X3" device=""/>
 <part name="JP8" library="adafruit" deviceset="PINHD-1X3" device=""/>
-<part name="L2" library="SparkFun-LED" deviceset="LED" device="5MM" value="Amber"/>
+<part name="L2" library="SparkFun-LED" deviceset="LED" device="5MM" value="Yellow"/>
 <part name="L3" library="SparkFun-LED" deviceset="LED" device="5MM" value="Green"/>
 <part name="L4" library="SparkFun-LED" deviceset="LED" device="5MM" value="Blue"/>
@@
 <part name="RB8" library="SparkFun-Resistors" deviceset="RESISTOR" device="0805-RES" value="100Ω"/>
 <part name="PF8" library="adafruit" deviceset="PINHD-1X1" device=""/>
-<part name="L5" library="SparkFun-LED" deviceset="LED" device="5MM" value="Yellow"/>
+<part name="L5" library="SparkFun-LED" deviceset="LED" device="5MM" value="Orange"/>
 <part name="OFF/ON" library="SparkFun-Electromechanical" deviceset="SWITCH-SPDT" device="KIT"/>
 <part name="RB11" library="SparkFun-Resistors" deviceset="RESISTOR" device="0805-RES" value="100Ω"/>

Commit message: Version 1 - 18th May 2023
Parts:
- L2: value Yellow -> Orange
- L5: value Orange -> Yellow
Changed lines of the file:
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@@
 <layer number="93" name="Pins" color="2" fill="1" visible="no" active="yes"/>
 <layer number="94" name="Symbols" color="4" fill="1" visible="yes" active="yes"/>
-<layer number="95" name="Names" color="7" fill="1" visible="no" active="yes"/>
+<layer number="95" name="Names" color="7" fill="1" visible="yes" active="yes"/>
 <layer number="96" name="Values" color="7" fill="1" visible="yes" active="yes"/>
 <layer number="97" name="Info" color="7" fill="1" visible="yes" active="yes"/>
@@
 <part name="JP7" library="adafruit" deviceset="PINHD-1X3" device=""/>
 <part name="JP8" library="adafruit" deviceset="PINHD-1X3" device=""/>
-<part name="L2" library="SparkFun-LED" deviceset="LED" device="5MM" value="Yellow"/>
+<part name="L2" library="SparkFun-LED" deviceset="LED" device="5MM" value="Orange"/>
 <part name="L3" library="SparkFun-LED" deviceset="LED" device="5MM" value="Green"/>
 <part name="L4" library="SparkFun-LED" deviceset="LED" device="5MM" value="Blue"/>
@@
 <part name="RB8" library="SparkFun-Resistors" deviceset="RESISTOR" device="0805-RES" value="100Ω"/>
 <part name="PF8" library="adafruit" deviceset="PINHD-1X1" device=""/>
-<part name="L5" library="SparkFun-LED" deviceset="LED" device="5MM" value="Orange"/>
+<part name="L5" library="SparkFun-LED" deviceset="LED" device="5MM" value="Yellow"/>
 <part name="OFF/ON" library="SparkFun-Electromechanical" deviceset="SWITCH-SPDT" device="KIT"/>
 <part name="RB11" library="SparkFun-Resistors" deviceset="RESISTOR" device="0805-RES" value="100Ω"/>
